File: kicad/led-candle.kicad_pcb (KiCad board)
At the start: 2 copper layers, 5 parts, among them J1 Conn_01x02, SW1 SW_SPDT, U1 ATtiny13A-P

Commit message: bugfix: fix a track in PCB
Routing:
- net GND: track 46.6 -> 48.1 mm
Changed lines of the file:
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@@
   (segment (start 147.1985 91.3185) (end 137.16 81.28) (width 0.25) (layer "B.Cu") (net 1))
   (segment (start 147.1985 104.14) (end 147.1985 91.3185) (width 0.25) (layer "B.Cu") (net 1))
-  (segment (start 157.47 91.43) (end 154.94 93.96) (width 0.25) (layer "B.Cu") (net 2))
-  (segment (start 137.16 109.22) (end 137.16 101.77) (width 0.25) (layer "B.Cu") (net 2))
-  (segment (start 154.94 93.96) (end 154.94 109.22) (width 0.25) (layer "B.Cu") (net 2))
+  (segment (start 154.95 91.43) (end 154.94 91.44) (width 0.25) (layer "B.Cu") (net 2))
+  (segment (start 157.47 91.43) (end 154.95 91.43) (width 0.25) (layer "B.Cu") (net 2))
   (segment (start 154.94 109.22) (end 137.16 109.22) (width 0.25) (layer "B.Cu") (net 2))
   (segment (start 157.48 88.9) (end 157.48 91.42) (width 0.25) (layer "B.Cu") (net 2))
   (segment (start 157.48 91.42) (end 157.47 91.43) (width 0.25) (layer "B.Cu") (net 2))
+  (segment (start 154.94 91.44) (end 154.94 109.22) (width 0.25) (layer "B.Cu") (net 2))
+  (segment (start 137.16 109.22) (end 137.16 101.77) (width 0.25) (layer "B.Cu") (net 2))
   (segment (start 149.86 86.36) (end 157.48 86.36) (width 0.25) (layer "B.Cu") (net 3))
   (segment (start 149.86 91.42) (end 149.85 91.43) (width 0.25) (layer "B.Cu") (net 4))
